Commit message: Stable conversion with simple friction model

File: finger_2r.urdf (robot description, URDF)
Before this commit: robot finger2r, 3 links, 2 joints
Joints:
- joint joint1: limit lower=-3.14 upper=3.14 effort=50 velocity=6.0 -> lower=-300.14 upper=300.14 effort=50 velocity=6.0
- joint joint2: limit lower=-3.14 upper=3.14 effort=50 velocity=6.0 -> lower=-300.14 upper=300.14 effort=50 velocity=6.0

Commit message: Bigger and heavier fingers

File: finger_2r.urdf (robot description, URDF)
Before this commit: robot finger2r, 3 links, 2 joints
Links:
- link link1: mass 0.5 -> M1; geometry collision box size=0.5 0.02 0.02; visual box size=0.5 0.02 0.02
- link link2: mass 0.01 -> M2; geometry collision box size=0.5 0.018 0.018; visual box size=0.5 0.018 0.018
Joints:
- joint joint2: origin xyz=0.15 0 0 rpy=0 0 0 -> xyz=0.5 0 0 rpy=0 0 0

Commit message: Pause on this branch

File: finger_2r.urdf (robot description, URDF)
Before this commit: robot finger2r, 3 links, 2 joints
Links:
- link link1: mass M1 -> 2.0; geometry collision box size=0.5 0.08 0.08; visual box size=0.5 0.08 0.08
- link link2: mass M2 -> 0.01; geometry collision box size=0.5 0.08 0.08; visual box size=0.5 0.08 0.08

Commit message: stable same trajectory in 2 joints but with diff friction

File: finger_2r.urdf (robot description, URDF)
Before this commit: robot finger2r, 2 links, 1 joints
Links:
- added link link2, mass 2.0; collision box size=0.5 0.07 0.07; visual box size=0.5 0.07 0.07
Joints:
- added joint joint2: type revolute, parent link1, child link2, origin xyz=0.5 0 0 rpy=0 0 0, axis 0 0 1, limit lower=-200.6 upper=200.6 effort=200 velocity=6.0
- joint joint1: limit lower=-300.14 upper=300.14 effort=50 velocity=6.0 -> lower=-200.6 upper=200.6 effort=200 velocity=6.0

Commit message: Fix some errors xD

File: finger_2r.urdf (robot description, URDF)
Before this commit: robot finger2r, 3 links, 2 joints
Joints:
- joint joint1: limit lower=-200.6 upper=200.6 effort=200 velocity=6.0 -> lower=-1.8 upper=1.8 effort=200 velocity=6.0
- joint joint2: limit lower=-200.6 upper=200.6 effort=200 velocity=6.0 -> lower=-1.8 upper=1.8 effort=200 velocity=6.0

Commit message: Ahaha

File: finger_2r.urdf (robot description, URDF)
Before this commit: robot finger2r, 3 links, 2 joints
Joints:
- joint joint1: limit lower=-1.8 upper=1.8 effort=200 velocity=6.0 -> lower=-100.8 upper=100.8 effort=200 velocity=6.0
- joint joint2: limit lower=-1.8 upper=1.8 effort=200 velocity=6.0 -> lower=-100.8 upper=100.8 effort=200 velocity=6.0
